File: power.kicad_sch (KiCad schematic)
At the start: 0 parts

Commit message: power and sd added
Parts:
- added C2, C4: 22 uF/10V, Capacitor_SMD:C_0603_1608Metric, symbol Device:C
- added D7: LED, LED_SMD:LED_0603_1608Metric, symbol Device:LED
- added R1: 2k, Resistor_SMD:R_0402_1005Metric, symbol Device:R
- added U3: AMS1117-3.3, Package_TO_SOT_SMD:SOT-223-3_TabPin2, symbol Regulator_Linear:AMS1117-3.3
Connections:
- new net: D7.2 (A), R1.2
- new net EXT_5V: C2.1, R1.1, U3.3 (VI)
- new net GND: C2.2, C4.2, D7.1 (K), U3.1 (GND)
- new net VDD33: C4.1, U3.2 (VO)
