File: sd_card.kicad_sch (KiCad schematic)
At the start: 7 parts, among them J4 Micro_SD_Card

Commit message: amp and sd sheets revision 1
Parts:
- C1: value C -> 100n; footprint (none) -> Capacitor_SMD:C_0603_1608Metric
- C3: value C -> 10u; footprint (none) -> Capacitor_SMD:C_0603_1608Metric
- J4: footprint (none) -> Connector_Card:microSD_HC_Hirose_DM3AT-SF-PEJM5
- R2, R3, R4, R5: value R -> 10k; footprint (none) -> Resistor_SMD:R_0402_1005Metric
Changed lines of the file:
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@@
 			)
 		)
-		(property "Value" "R"
+		(property "Value" "10k"
 			(at 142.24 58.4199 0)
 			(effects
@@
 			)
 		)
-		(property "Footprint" ""
+		(property "Footprint" "Resistor_SMD:R_0402_1005Metric"
 			(at 137.922 57.15 90)
 			(effects
@@
 			)
 		)
-		(property "Value" "C"
+		(property "Value" "100n"
 			(at 118.11 93.9799 0)
 			(effects
@@
 			)
 		)
-		(property "Footprint" ""
+		(property "Footprint" "Capacitor_SMD:C_0603_1608Metric"
 			(at 115.2652 96.52 0)
 			(effects
@@
 			)
 		)
-		(property "Value" "C"
+		(property "Value" "10u"
 			(at 130.81 93.9799 0)
 			(effects
@@
 			)
 		)
-		(property "Footprint" ""
+		(property "Footprint" "Capacitor_SMD:C_0603_1608Metric"
 			(at 127.9652 96.52 0)
 			(effects
@@
 			)
 		)
-		(property "Value" "R"
+		(property "Value" "10k"
 			(at 154.94 58.4199 0)
 			(effects
@@
 			)
 		)
-		(property "Footprint" ""
+		(property "Footprint" "Resistor_SMD:R_0402_1005Metric"
 			(at 150.622 57.15 90)
 			(effects
@@
 			)
 		)
-		(property "Value" "R"
+		(property "Value" "10k"
 			(at 129.54 58.4199 0)
 			(effects
@@
 			)
 		)
-		(property "Footprint" ""
+		(property "Footprint" "Resistor_SMD:R_0402_1005Metric"
 			(at 125.222 57.15 90)
 			(effects
@@
 			)
 		)
-		(property "Value" "R"
+		(property "Value" "10k"
 			(at 116.84 58.4199 0)
 			(effects
@@
 			)
 		)
-		(property "Footprint" ""
+		(property "Footprint" "Resistor_SMD:R_0402_1005Metric"
 			(at 112.522 57.15 90)
 			(effects
@@
 				)
 				(hide yes)
+			)
+		)
+		(property "Purpose" ""
+			(at 114.3 57.15 0)
+			(effects
+				(font
+					(size 1.27 1.27)
+				)
 			)
 		)
@@
 			)
 		)
-		(property "Footprint" ""
+		(property "Footprint" "Connector_Card:microSD_HC_Hirose_DM3AT-SF-PEJM5"
 			(at 53.34 69.85 0)
 			(effects

Commit message: rfid revision 1 sch
Other:
- company: (none) -> C. Boerner
- title: (none) -> SD Card Module
Changed lines of the file:
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@@
 	(generator_version "9.0")
 	(paper "A4")
+	(title_block
+		(title "SD Card Module")
+		(date "2025-07-22")
+		(rev "1.0")
+		(company "C. Boerner")
+	)
 	(junction
 		(at 127 74.93)
