File: 1.Hardware/rfid.kicad_sch (KiCad schematic)
At the start: 31 parts, among them Q3 2N7002, Q4 2N7002, U3 PN5321A3HN_C1xx, Y1 27.12MHz

Commit message: updated schematic to match demo
Parts:
- C12, C13, C2, C24, C31, C32: value C -> 0.1u
- C23: value C -> 4.7u
- C25, C26: value C -> 220p
- C27, C28, C34, C35: value C -> 22p
- C29, C30: value C -> 200p
- C33: value C -> 1n
- C4: value C -> 10u
- L1, L2: value L -> 560n
- R1: value R -> 10k
- R10: value R -> 1.6k
- R14, R15: value R -> 4.7k
- R6: value R -> 20k
- R9: value R -> 1k
Connections:
- net RXD: now also Q4.3 (D); no longer Q3.3 (D)
- net TXD: now also Q3.3 (D); no longer Q4.3 (D)
Changed lines of the file:
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@@
 		)
 	)
-	(hierarchical_label "TXD"
+	(hierarchical_label "RXD"
 		(shape input)
 		(at 215.9 101.6 0)
@@
 		)
 	)
-	(hierarchical_label "RXD"
+	(hierarchical_label "TXD"
 		(shape input)
 		(at 215.9 76.2 0)
@@
 			)
 		)
-		(property "Value" "C"
-			(at 167.64 113.03 0)
+		(property "Value" "0.1u"
+			(at 166.878 115.824 0)
 			(effects
 				(font
@@
 			)
 		)
-		(property "Value" "R"
+		(property "Value" "1k"
 			(at 105.41 107.95 0)
 			(effects
@@
 			)
 		)
-		(property "Value" "C"
-			(at 105.41 124.46 0)
+		(property "Value" "0.1u"
+			(at 104.394 127 0)
 			(effects
 				(font
@@
 		(dnp no)
 		(property "Reference" "C32"
-			(at 96.52 106.68 0)
-			(effects
-				(font
-					(size 1.27 1.27)
-				)
-				(justify left)
-			)
-		)
-		(property "Value" "C"
-			(at 99.06 106.68 0)
+			(at 100.584 99.314 90)
+			(effects
+				(font
+					(size 1.27 1.27)
+				)
+				(justify left)
+			)
+		)
+		(property "Value" "0.1u"
+			(at 99.568 106.172 90)
 			(effects
 				(font
@@
 		(dnp no)
 		(property "Reference" "C30"
-			(at 74.93 95.25 0)
-			(effects
-				(font
-					(size 1.27 1.27)
-				)
-				(justify left)
-			)
-		)
-		(property "Value" "C"
-			(at 73.66 92.71 0)
+			(at 66.802 91.44 0)
+			(effects
+				(font
+					(size 1.27 1.27)
+				)
+				(justify left)
+			)
+		)
+		(property "Value" "200p"
+			(at 66.802 93.726 0)
 			(effects
 				(font
@@
 			)
 		)
-		(property "Value" "L"
+		(property "Value" "560n"
 			(at 99.06 88.9 90)
 			(effects
@@
 			)
 		)
-		(property "Value" "R"
+		(property "Value" "4.7k"
 			(at 193.04 72.3899 0)
 			(effects
@@
 			)
 		)
-		(property "Value" "C"
-			(at 120.65 138.43 0)
+		(property "Value" "22p"
+			(at 120.142 141.224 0)
 			(effects
 				(font
@@
 			)
 		)
-		(property "Value" "C"
-			(at 110.49 43.18 0)
+		(property "Value" "0.1u"
+			(at 109.22 45.72 0)
 			(effects
 				(font
@@
 		(dnp no)
 		(property "Reference" "C28"
-			(at 76.2 101.6 0)
-			(effects
-				(font
-					(size 1.27 1.27)
-				)
-				(justify left)
-			)
-		)
-		(property "Value" "C"
-			(at 78.74 100.33 0)
+			(at 80.01 92.964 90)
+			(effects
+				(font
+					(size 1.27 1.27)
+				)
+				(justify left)
+			)
+		)
+		(property "Value" "22p"
+			(at 80.518 100.838 90)
 			(effects
 				(font
@@
 		(dnp no)
 		(property "Reference" "C2"
-			(at 107.95 54.61 0)
-			(effects
-				(font
-					(size 1.27 1.27)
-				)
-				(justify left)
-			)
-		)
-		(property "Value" "C"
-			(at 109.22 57.15 0)
+			(at 109.728 54.864 0)
+			(effects
+				(font
+					(size 1.27 1.27)
+				)
+				(justify left)
+			)
+		)
+		(property "Value" "0.1u"
+			(at 109.22 59.436 0)
 			(effects
 				(font
@@
 			)
 		)
-		(property "Value" "L"
+		(property "Value" "560n"
 			(at 99.06 81.28 90)
 			(effects
@@
 			)
 		)
-		(property "Value" "R"
+		(property "Value" "10k"
 			(at 135.89 43.1799 0)
 			(effects
@@
 		(dnp no)
 		(property "Reference" "R10"
-			(at 87.63 110.49 0)
+			(at 90.932 109.22 90)
 			(effects
 				(font
@@
 			)
 		)
-		(property "Value" "R"
-			(at 90.17 110.49 0)
+		(property "Value" "1.6k"
+			(at 90.932 114.554 90)
 			(effects
 				(font
@@
 			)
 		)
-		(property "Value" "C"
-			(at 83.82 92.71 0)
+		(property "Value" "220p"
+			(at 82.042 94.996 0)
 			(effects
 				(font
@@
 			)
 		)
-		(property "Value" "C"
-			(at 83.82 82.55 0)
+		(property "Value" "220p"
+			(at 82.296 84.836 0)
 			(effects
 				(font
@@
 		(dnp no)
 		(property "Reference" "C35"
-			(at 148.59 135.89 0)
-			(effects
-				(font
-					(size 1.27 1.27)
-				)
-				(justify left)
-			)
-		)
-		(property "Value" "C"
-			(at 148.59 138.43 0)
+			(at 153.416 135.636 0)
+			(effects
+				(font
+					(size 1.27 1.27)
+				)
+				(justify left)
+			)
+		)
+		(property "Value" "22p"
+			(at 152.908 141.224 0)
 			(effects
 				(font
@@
 		(dnp no)
 		(property "Reference" "C27"
-			(at 76.2 82.55 0)
-			(effects
-				(font
-					(size 1.27 1.27)
-				)
-				(justify left)
-			)
-		)
-		(property "Value" "C"
-			(at 78.74 81.28 0)
+			(at 80.518 73.914 90)
+			(effects
+				(font
+					(size 1.27 1.27)
+				)
+				(justify left)
+			)
+		)
+		(property "Value" "22p"
+			(at 80.772 81.026 90)
 			(effects
 				(font
@@
 		(dnp no)
 		(property "Reference" "C29"
-			(at 74.93 85.09 0)
-			(effects
-				(font
-					(size 1.27 1.27)
-				)
-				(justify left)
-			)
-		)
-		(property "Value" "C"
-			(at 73.66 82.55 0)
+			(at 66.802 80.518 0)
+			(effects
+				(font
+					(size 1.27 1.27)
+				)
+				(justify left)
+			)
+		)
+		(property "Value" "200p"
+			(at 67.564 82.55 0)
 			(effects
 				(font
@@
 		)
 		(property "Value" "100"
-			(at 170.18 101.6 90)
+			(at 170.18 104.394 90)
 			(effects
 				(font
@@
 			)
 		)
-		(property "Value" "C"
-			(at 118.11 43.18 0)
+		(property "Value" "10u"
+			(at 117.602 45.974 0)
 			(effects
 				(font
@@
 			)
 		)
-		(property "Value" "C"
-			(at 90.17 68.58 0)
+		(property "Value" "0.1u"
+			(at 88.9 71.12 0)
 			(effects
 				(font
@@
 		(dnp no)
 		(property "Reference" "C33"
-			(at 96.52 115.57 0)
-			(effects
-				(font
-					(size 1.27 1.27)
-				)
-				(justify left)
-			)
-		)
-		(property "Value" "C"
-			(at 99.06 115.57 0)
+			(at 100.584 108.458 90)
+			(effects
+				(font
+					(size 1.27 1.27)
+				)
+				(justify left)
+			)
+		)
+		(property "Value" "1n"
+			(at 100.33 115.062 90)
 			(effects
 				(font
@@
 			)
 		)
-		(property "Value" "R"
+		(property "Value" "4.7k"
 			(at 193.04 97.7899 0)
 			(effects
@@
 			)
 		)
-		(property "Value" "C"
-			(at 97.79 68.58 0)
+		(property "Value" "4.7u"
+			(at 96.774 71.374 0)
 			(effects
 				(font
@@
 			)
 		)
-		(property "Value" "R"
+		(property "Value" "20k"
 			(at 135.89 52.0699 0)
 			(effects

Commit message: ready for routing/placement
Parts:
- removed R16: 100, symbol Device:R
Connections:
- net RSTOUT: no longer names the net of U3.26 (~{RSTOUT})
- no-connect marks 14 -> 16
Changed lines of the file:
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@@
 	)
 	(no_connect
+		(at 165.1 101.6)
+	)
+	(no_connect
 		(at 128.27 118.11)
 	)
@@
 	)
 	(no_connect
+		(at 165.1 97.79)
+	)
+	(no_connect
 		(at 165.1 86.36)
 	)
@@
 	(wire
 		(pts
-			(xy 165.1 97.79) (xy 173.99 97.79)
-		)
-		(stroke
-			(width 0)
-			(type default)
-		)
-	)
-	(wire
-		(pts
 			(xy 105.41 63.5) (xy 101.6 63.5)
 		)
@@
 	(wire
 		(pts
-			(xy 165.1 101.6) (xy 166.37 101.6)
-		)
-		(stroke
-			(width 0)
-			(type default)
-		)
-	)
-	(wire
-		(pts
 			(xy 124.46 118.11) (xy 124.46 120.65)
 		)
@@
 		)
 	)
+	(label "RXD"
+		(at 215.9 101.6 0)
+		(effects
+			(font
+				(size 1.27 1.27)
+			)
+			(justify left bottom)
+		)
+	)
+	(label "TXD"
+		(at 215.9 76.2 0)
+		(effects
+			(font
+				(size 1.27 1.27)
+			)
+			(justify left bottom)
+		)
+	)
 	(global_label "VDD33"
 		(shape input)
@@
 		)
 	)
-	(hierarchical_label "RSTOUT"
-		(shape input)
-		(at 173.99 97.79 0)
-		(effects
-			(font
-				(size 1.27 1.27)
-			)
-			(justify left)
-		)
-	)
-	(hierarchical_label "RXD"
-		(shape input)
-		(at 215.9 101.6 0)
-		(effects
-			(font
-				(size 1.27 1.27)
-			)
-			(justify left)
-		)
-	)
-	(hierarchical_label "TXD"
-		(shape input)
-		(at 215.9 76.2 0)
-		(effects
-			(font
-				(size 1.27 1.27)
-			)
-			(justify left)
-		)
-	)
-	(hierarchical_label "IRQ"
-		(shape input)
-		(at 173.99 101.6 0)
-		(effects
-			(font
-				(size 1.27 1.27)
-			)
-			(justify left)
-		)
-	)
 	(symbol
 		(lib_id "Device:C")
@@
 					(unit 1)
 				)
-			)
-		)
-	)
-	(symbol
-		(lib_id "Device:R")
-		(at 170.18 101.6 270)
-		(unit 1)
-		(exclude_from_sim no)
-		(in_bom yes)
-		(on_board yes)
-		(dnp no)
-		(property "Reference" "R16"
-			(at 170.18 99.06 90)
-			(effects
-				(font
-					(size 1.27 1.27)
-				)
-			)
-		)
-		(property "Value" "100"
-			(at 170.18 104.394 90)
-			(effects
-				(font
-					(size 1.27 1.27)
-				)
-			)
-		)
-		(property "Footprint" ""
-			(at 170.18 99.822 90)
-			(effects
-				(font
-					(size 1.27 1.27)
-				)
-				(hide yes)
-			)
-		)
-		(property "Datasheet" "~"
-			(at 170.18 101.6 0)
-			(effects
-				(font
-					(size 1.27 1.27)
-				)
-				(hide yes)
-			)
-		)
-		(property "Description" "Resistor"
-			(at 170.18 101.6 0)
-			(effects
-				(font
-					(size 1.27 1.27)
-				)
-				(hide yes)
-			)
-		)
-		(pin "2"
-		)
-		(pin "1"
-		)
-		(instances
-			(project "jukebox"
-				(path "/d400bd10-35e9-4717-b347-ccb991be6072/c6b3536d-842a-485c-ace2-2998012aef86"
-					(reference "R16")
-					(unit 1)
-				)
